File: hardware/PCB/Mezmerize_B1_Controller.kicad_sch (KiCad schematic)
At the start: 47 parts, among them J1 230 Vac, J10 I2C DISPLAY (OLED/LCD), J11 I2C (FUTURE USE), J12 ROTARY ENC & SWITCH (FUTURE U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, J13 ROTARY ENC & SWITCH, J14 IR RECV, J2 B1 Relays, J3 PWR AMP L 12V TRIGGER, J4 PWR AMP L SWITCH, J5 PWR AMP R 12V TRIGGER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

Commit message: Schematic cleanup
Parts:
- U8: value (none) -> ESP32-DEVKIT-V1; footprint (none) -> MODULE_ESP32_DEVKIT_V1
Connections:
- net NTC_R: no longer J9.5 (Pin_5), U8.10 (D19)
- new net: J9.5 (Pin_5), U8.10 (D19)
- no-connect marks 7 -> 15
Other:
- moved on the sheet: J7, J8, R5, R6, R7, R8, U8
