File: hardware/PCB/Mezmerize_B1_Controller.kicad_sch (KiCad schematic)
At the start: 48 parts, among them J1 230 Vac, J10 I2C DISPLAY (OLED/LCD), J11 I2C (FUTURE USE), J12 ROTARY ENC & SWITCH 1, J13 ROTARY ENC & SWITCH 2, J14 IR RECV, J2 B1 Relays, J3 PWR AMP L 12V TRIGGER, J4 PWR AMP L SWITCH, J5 PWR AMP R 12V TRIGGER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

Commit message: Update to new esp32 symbol
Parts:
- removed U8: ESP32-DEVKIT-V1, MODULE_ESP32_DEVKIT_V1, symbol ESP32:ESP32-DEVKIT-V1
- U?: value (none) -> ESP32-DEVKIT-V1; footprint (none) -> MODULE_ESP32_DEVKIT_V1
Connections:
- net +3V3: now also U?.1 (3V3)
- net +8V: now also U?.30 (VIN)
- net CCW_1: now also U?.24 (D26)
- net CCW_2: now also U?.27 (D12)
- net CONTRAST(LCD): now also U?.22 (D33)
- net CW_1: now also U?.23 (D25)
- net CW_2: now also U?.26 (D14)
- net GND: now also U?.29 (GND)
- net I2C:SCL: now also U?.14 (D22); no longer R6.1
- net I2C:SDA: now also U?.11 (D21)
- net IR OUT: now also U?.21 (D32)
- net L_MEASURE_ON_OFF: now also U?.5 (D4)
- net NTC_L: now also U?.20 (D35)
- net NTC_R: now also U?.19 (D34)
- net R_MEASURE_ON_OFF: now also U?.3 (D15)
- net SPI:MISO: now also U?.10 (D19)
- net SPI:MOSI: now also R6.1, U?.15 (D23)
- net SPI:SCK: now also U?.9 (D18)
- net SPI:SS: now also U?.8 (D5)
- net SW_1: now also U?.25 (D27)
- net SW_2: now also U?.28 (D13)
- no-connect marks 15 -> 11
Other:
- moved on the sheet: R5, R6, U?
