File: hardware/Power Supply/Power Supply.kicad_sch (KiCad schematic)
At the start: 17 parts, among them J1 230 Vac, U4 L7808CV

Commit message: psu pcb ready
Parts:
- J2: value (none) -> 12V
- J3: value (none) -> 8V
Connections:
- net at F2.2, PS1.1 (AC/L), RV1.1: no longer F1.2, F2.1
- new net: F1.2, F2.1
Changed lines of the file:
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@@
   (junction (at 214.63 80.01) (diameter 0) (color 0 0 0 0)
   )
-  (junction (at 107.95 80.01) (diameter 0) (color 0 0 0 0)
-  )
   (junction (at 163.83 80.01) (diameter 0) (color 0 0 0 0)
   )
@@
   (junction (at 182.88 80.01) (diameter 0) (color 0 0 0 0)
   )
-  (junction (at 107.95 72.39) (diameter 0) (color 0 0 0 0)
-  )
   (junction (at 142.24 80.01) (diameter 0) (color 0 0 0 0)
   )
@@
   )
   (wire (pts (xy 107.95 80.01) (xy 113.03 80.01))
-    (stroke (width 0) (type default) (color 0 0 0 0))
-  )
-  (wire (pts (xy 107.95 72.39) (xy 107.95 80.01))
     (stroke (width 0) (type default) (color 0 0 0 0))
   )
@@
       (effects (font (size 1.27 1.27)) hide)
     )
-    (property "Value" "" (id 1) (at 202.5651 57.5838 90)
+    (property "Value" "GND" (id 1) (at 202.5651 57.5838 90)
       (effects (font (size 1.27 1.27)) (justify right))
     )
@@
       (effects (font (size 1.27 1.27)) hide)
     )
-    (property "Value" "" (id 1) (at 153.0366 55.88 0))
+    (property "Value" "GND" (id 1) (at 153.0366 55.88 0))
     (property "Footprint" "" (id 2) (at 157.48 55.88 0)
       (effects (font (size 1.27 1.27)) hide)
@@
     (in_bom yes) (on_board yes)
     (property "Reference" "J3" (id 0) (at 220.345 54.1528 0))
-    (property "Value" "" (id 1) (at 218.0336 54.1528 0))
+    (property "Value" "8V" (id 1) (at 218.0336 54.1528 0))
     (property "Footprint" "TerminalBlock:TerminalBlock_bornier-2_P5.08mm" (id 2) (at 212.09 52.07 0)
       (effects (font (size 1.27 1.27)) hide)
@@
     (in_bom yes) (on_board yes)
     (property "Reference" "J2" (id 0) (at 169.545 52.8828 0))
-    (property "Value" "" (id 1) (at 167.2336 52.8828 0))
+    (property "Value" "12V" (id 1) (at 167.2336 52.8828 0))
     (property "Footprint" "TerminalBlock:TerminalBlock_bornier-2_P5.08mm" (id 2) (at 161.29 50.8 0)
       (effects (font (size 1.27 1.27)) hide)
